File: hardware/BeeLight.kicad_pcb (KiCad board)
At the start: 2 copper layers, 32 x 24 mm, 25 parts, among them IC102 APDS-9306-065, IC103 BME688, M101 BL54L15, Q101 BSS84, SW101 JOIN, X102 DEBUG

Commit message: Some weird errors
Parts:
- R109: value 2k2 -> 1k
- moved X102 8.71 mm to (150.4, 93.2)
